Commit message: modified to appear tf in rviz2

File: aiformula_description/urdf/ai_car.urdf (robot description, URDF)
Before this commit: robot ai_car, 5 links, 4 joints
Links:
- removed link caster_link
- removed link left_wheel_link
- removed link right_wheel_link
- added link camera_depth_frame
- added link camera_depth_optical_frame
- added link camera_link; collision box size=0.012 0.132 0.020; visual mesh filename=package://aiformula_description/meshes/r200.dae
- added link camera_rgb_frame
- added link camera_rgb_optical_frame
- added link caster_back_link, mass 0.005; collision box size=0.030 0.009 0.020; visual mesh filename=package://aiformula_description/meshes/tire_v1.dae scale=0.1 0.1 0.1
- added link imu_link
- added link wheel_left_link, mass 7.0; collision mesh filename=package://aiformula_description/meshes/tire_v1.dae scale=0.05 0.12 0.12; visual mesh filename=package://aiformula_description/meshes/tire_v1.dae scale=0.05 0.12 0.12
- added link wheel_right_link, mass 7.0; collision mesh filename=package://aiformula_description/meshes/tire_v1.dae scale=0.05 0.12 0.12; visual mesh filename=package://aiformula_description/meshes/tire_v1.dae scale=0.05 0.12 0.12
- link base_link: mass 30.0 -> 30
Joints:
- removed joint caster_wheel_joint
- removed joint left_wheel_joint
- removed joint right_wheel_joint
- added joint camera_depth_joint: type fixed, parent camera_link, child camera_depth_frame, origin xyz=0.005 0.028 0.013 rpy=0 0 0
- added joint camera_depth_optical_joint: type fixed, parent camera_depth_frame, child camera_depth_optical_frame, origin xyz=0 0 0 rpy=-1.57 0 -1.57
- added joint camera_joint: type fixed, parent base_link, child camera_link, origin xyz=0.064 -0.065 0.44 rpy=0 0 0
- added joint camera_rgb_joint: type fixed, parent camera_link, child camera_rgb_frame, origin xyz=0.005 0.018 0.013 rpy=0 0 0
- added joint camera_rgb_optical_joint: type fixed, parent camera_rgb_frame, child camera_rgb_optical_frame, origin xyz=0 0 0 rpy=-1.57 0 -1.57
- added joint caster_back_joint: type fixed, parent base_link, child caster_back_link, origin xyz=-0.85 0.0 0.0 rpy=1.57 0 1.57
- added joint imu_joint: type fixed, parent base_link, child imu_link, origin xyz=0.0 0 0.068 rpy=0 0 0
- added joint wheel_left_joint: type continuous, parent base_link, child wheel_left_link, origin xyz=0.0 0.3 0.0 rpy=1.57 0 1.57, axis 1 0 0
- added joint wheel_right_joint: type continuous, parent base_link, child wheel_right_link, origin xyz=0.0 -0.3 0.0 rpy=1.57 0 1.57, axis 1 0 0
- joint base_joint: origin xyz=0 0 0.15 rpy=0 0 0 -> xyz=0 0 0.010 rpy=0 0 0
