Commit message: Delete unnecessary files related to xacro

File: vehicle/xacro/parts/caster_back_macro.xacro (robot description, xacro)
@@ -14,5 +14,5 @@
                params="caster_back
                        x y z roll pitch yaw">
-    <xacro:property name="MESH_FILE" value="package://vehicle/xacro/meshes/tire_v1.dae"/>
+    <xacro:property name="MESH_FILE" value="package://vehicle/xacro/meshes/tire.dae"/>
     <xacro:property name="SCALE" value="0.10"/>
     <link name="${caster_back}_link">

File: vehicle/xacro/parts/wheel_macro.xacro (robot description, xacro)
@@ -14,5 +14,5 @@
                params="wheel
                        x y z roll pitch yaw">
-    <xacro:property name="MESH_FILE" value="package://vehicle/xacro/meshes/tire_v1.dae"/>
+    <xacro:property name="MESH_FILE" value="package://vehicle/xacro/meshes/tire.dae"/>
     <xacro:property name="THICKNESS_SCALE" value="0.05"/>
     <xacro:property name="SIZE_SCALE" value="0.12"/>

File: vehicle/xacro/parts/zed_macro.xacro (robot description, xacro)
@@ -13,5 +13,5 @@
                params="camera
                        size_x size_y size_z roll pitch yaw">
-    <xacro:property name="MESH_FILE" value="package://vehicle/xacro/meshes/r200.dae"/>
+    <xacro:property name="MESH_FILE" value="package://vehicle/xacro/meshes/realsense_r200.dae"/>
     <link name="${camera}_link">
       <visual>
