Commit message: Correct spelling errors and add const qualifier to pointers.

File: vehicle/xacro/parts/zed_macro.xacro (robot description, xacro)
@@ -4,5 +4,5 @@
                params="camera parent zed_serial_number">
     <xacro:property name="ZED_PARAM_YAML_PATH" value="$(find vehicle)/config/zedx/camera_params/${zed_serial_number}/extrinsic.yaml" />
-    <xacro:property name="POSISION" value="${load_yaml(ZED_PARAM_YAML_PATH)['position']}" />
+    <xacro:property name="POSITION" value="${load_yaml(ZED_PARAM_YAML_PATH)['position']}" />
     <xacro:property name="ORIENTATION" value="${load_yaml(ZED_PARAM_YAML_PATH)['orientation']}" />
     <xacro:property name="MESH_FILE" value="package://vehicle/xacro/meshes/zedx.stl"/>
@@ -12,5 +12,5 @@
       <parent link="${parent}_link"/>
       <child  link="${camera}_camera_link"/>
-      <origin xyz="${POSISION['x']} ${POSISION['y']} ${POSISION['z']}" rpy="0.0  0.0  0.0"/>
+      <origin xyz="${POSITION['x']} ${POSITION['y']} ${POSITION['z']}" rpy="0.0  0.0  0.0"/>
     </joint>
     <link name="${camera}_camera_link" />
