Commit message: Correct installation angle of zedX

File: vehicle/xacro/ai_car1.xacro (robot description, xacro)
@@ -9,50 +9,50 @@
   <xacro:property name="WHEEL_RADIUS" value="0.12"/>
   <xacro:property name="CASTER_RADIUS" value="0.10"/>
-  <xacro:property name="base_footprint" value="base_footprint"/>
-  <xacro:property name="base" value="base"/>
-  <xacro:property name="wheel_left" value="wheel_left"/>
-  <xacro:property name="wheel_right" value="wheel_right"/>
-  <xacro:property name="caster_back" value="caster_back"/>
-  <xacro:property name="zedX" value="zedX"/>
+  <xacro:property name="BASE_FOOTPRINT" value="base_footprint"/>
+  <xacro:property name="BASE" value="base"/>
+  <xacro:property name="ZEDX" value="zedX"/>
+  <xacro:property name="WHEEL_LEFT" value="wheel_left"/>
+  <xacro:property name="WHEEL_RIGHT" value="wheel_right"/>
+  <xacro:property name="CASTER_BACK" value="caster_back"/>
   <!-- base_footprint -->
-  <link name="${base_footprint}"/>
+  <link name="${BASE_FOOTPRINT}"/>
   <!-- base -->
   <xacro:base_macro
-    base="${base}" parent_link="${base_footprint}"
+    base="${BASE}" parent_link="${BASE_FOOTPRINT}"
     x="0.0" y="0.0" z="${WHEEL_RADIUS}"
     roll="0.0" pitch="0.0" yaw="${180.0*D2R}"/>
   <!-- zedX -->
   <xacro:zed_joint_macro
-    camera="${zedX}" parent="${base}"
+    camera="${ZEDX}" parent="${BASE}"
     x="0.055" y="0.0" z="0.54"
-    roll="0.0" pitch="${2.0*D2R}" yaw="0.0"/>
+    roll="${(-90.0-2.0)*D2R}" pitch="0.0" yaw="${-90.0*D2R}"/>
   <xacro:zed_link_macro
-    camera="${zedX}"
-    size_x="0.006" size_y="0.132" size_z="0.020"
-    roll="${90.0*D2R}" pitch="0.0" yaw="${90.0*D2R}"/>
+    camera="${ZEDX}"
+    size_x="0.132" size_y="0.020" size_z="0.006"
+    roll="0.0" pitch="0.0" yaw="0.0"/>
   <!-- wheel -->
   <xacro:wheel_joint_macro
-    wheel="${wheel_left}" parent="${base}"
+    wheel="${WHEEL_LEFT}" parent="${BASE}"
     x="0.0" y="0.3" z="${WHEEL_RADIUS}"
     roll="${90.0*D2R}" pitch="0.0" yaw="${90.0*D2R}"/>
   <xacro:wheel_link_macro
-    wheel="${wheel_left}"
+    wheel="${WHEEL_LEFT}"
     x="0.0" y="0.0" z="0.0"
     roll="0.0" pitch="0.0" yaw="0.0"/>
   <xacro:wheel_joint_macro
-    wheel="${wheel_right}" parent="${base}"
+    wheel="${WHEEL_RIGHT}" parent="${BASE}"
     x="0.0" y="-0.3" z="${WHEEL_RADIUS}"
     roll="${90.0*D2R}" pitch="0.0" yaw="${90.0*D2R}"/>
   <xacro:wheel_link_macro
-    wheel="${wheel_right}"
+    wheel="${WHEEL_RIGHT}"
     x="0.0" y="0.0" z="0.0"
     roll="0.0" pitch="0.0" yaw="0.0"/>
   <!-- caster_back -->
   <xacro:caster_back_joint_macro
-    caster_back="${caster_back}" parent="${base}"
+    caster_back="${CASTER_BACK}" parent="${BASE}"
     x="-0.76" y="0.0" z="${CASTER_RADIUS}"
     roll="${90.0*D2R}" pitch="0.0" yaw="${90.0*D2R}"/>
   <xacro:caster_back_link_macro
-    caster_back="${caster_back}"
+    caster_back="${CASTER_BACK}"
     x="0.0" y="0.0" z="0.0"
     roll="0.0" pitch="0.0" yaw="0.0"/>

File: vehicle/xacro/parts/base.xacro (robot description, xacro)
@@ -9,10 +9,10 @@
       <origin xyz="0.0  0.0  0.0" rpy="0.0  0.0  0.0"/>
     </joint>
-    <xacro:property name="mesh_file" value="package://vehicle/xacro/meshes/AIF_body.dae"/>
+    <xacro:property name="MESH_FILE" value="package://vehicle/xacro/meshes/AIF_body.dae"/>
     <link name="${base}_link">
       <visual>
         <origin xyz="${x} ${y} ${z}" rpy="${roll} ${pitch} ${yaw}"/>
         <geometry>
-          <mesh filename="${mesh_file}"/>
+          <mesh filename="${MESH_FILE}"/>
         </geometry>
       </visual>
@@ -20,5 +20,5 @@
         <origin xyz="${x} ${y} ${z}" rpy="${roll} ${pitch} ${yaw}"/>
         <geometry>
-          <mesh filename="${mesh_file}"/>
+          <mesh filename="${MESH_FILE}"/>
         </geometry>
       </collision>

File: vehicle/xacro/parts/caster_back_macro.xacro (robot description, xacro)
@@ -14,11 +14,11 @@
                params="caster_back
                        x y z roll pitch yaw">
-    <xacro:property name="mesh_file" value="package://vehicle/xacro/meshes/tire_v1.dae"/>
-    <xacro:property name="scale" value="0.10"/>
+    <xacro:property name="MESH_FILE" value="package://vehicle/xacro/meshes/tire_v1.dae"/>
+    <xacro:property name="SCALE" value="0.10"/>
     <link name="${caster_back}_link">
       <visual>
         <origin xyz="${x} ${y} ${z}" rpy="${roll} ${pitch} ${yaw}"/>
         <geometry>
-          <mesh filename="${mesh_file}" scale="${scale} ${scale} ${scale}"/>
+          <mesh filename="${MESH_FILE}" scale="${SCALE} ${SCALE} ${SCALE}"/>
         </geometry>
       </visual>
@@ -26,5 +26,5 @@
         <origin xyz="${x} ${y} ${z}" rpy="${roll} ${pitch} ${yaw}"/>
         <geometry>
-          <mesh filename="${mesh_file}" scale="${scale} ${scale} ${scale}"/>
+          <mesh filename="${MESH_FILE}" scale="${SCALE} ${SCALE} ${SCALE}"/>
         </geometry>
         <!-- <origin xyz="0.0  0.001  0.0" rpy="0.0  0.0  0.0"/>

File: vehicle/xacro/parts/wheel_macro.xacro (robot description, xacro)
@@ -14,12 +14,12 @@
                params="wheel
                        x y z roll pitch yaw">
-    <xacro:property name="mesh_file" value="package://vehicle/xacro/meshes/tire_v1.dae"/>
-    <xacro:property name="thickness_scale" value="0.05"/>
-    <xacro:property name="size_scale" value="0.12"/>
+    <xacro:property name="MESH_FILE" value="package://vehicle/xacro/meshes/tire_v1.dae"/>
+    <xacro:property name="THICKNESS_SCALE" value="0.05"/>
+    <xacro:property name="SIZE_SCALE" value="0.12"/>
     <link name="${wheel}_link">
       <visual>
         <origin xyz="${x} ${y} ${z}" rpy="${roll} ${pitch} ${yaw}"/>
         <geometry>
-          <mesh filename="${mesh_file}" scale="${thickness_scale} ${size_scale} ${size_scale}"/>
+          <mesh filename="${MESH_FILE}" scale="${THICKNESS_SCALE} ${SIZE_SCALE} ${SIZE_SCALE}"/>
         </geometry>
       </visual>
@@ -27,5 +27,5 @@
         <origin xyz="${x} ${y} ${z}" rpy="${roll} ${pitch} ${yaw}"/>
         <geometry>
-          <mesh filename="${mesh_file}" scale="${thickness_scale} ${size_scale} ${size_scale}"/>
+          <mesh filename="${MESH_FILE}" scale="${THICKNESS_SCALE} ${SIZE_SCALE} ${SIZE_SCALE}"/>
         </geometry>
       </collision>

File: vehicle/xacro/parts/zed_macro.xacro (robot description, xacro)
@@ -13,10 +13,10 @@
                params="camera
                        size_x size_y size_z roll pitch yaw">
-    <xacro:property name="mesh_file" value="package://vehicle/xacro/meshes/r200.dae"/>
+    <xacro:property name="MESH_FILE" value="package://vehicle/xacro/meshes/r200.dae"/>
     <link name="${camera}_link">
       <visual>
         <origin xyz="${-size_x*0.5} ${-size_y*0.5} ${-size_z*0.5}" rpy="${roll} ${pitch} ${yaw}"/>
         <geometry>
-          <mesh filename="${mesh_file}"/>
+          <mesh filename="${MESH_FILE}"/>
         </geometry>
       </visual>
@@ -28,8 +28,9 @@
       </collision>
     </link>
+    <xacro:property name="BASE_LINE" value="0.120005"/>
     <joint name="${camera}_left_joint" type="fixed">
       <parent link="${camera}_link"/>
       <child link="${camera}_left_link"/>
-      <origin xyz="0.0 ${size_y*0.5} 0.0" rpy="0.0  0.0  0.0"/>
+      <origin xyz="${-BASE_LINE*0.5}  0.0  0.0" rpy="0.0  0.0  0.0"/>
     </joint>
     <link name="${camera}_left_link"/>
@@ -37,5 +38,5 @@
       <parent link="${camera}_link"/>
       <child link="${camera}_right_link"/>
-      <origin xyz="0.0 ${-size_y*0.5} 0.0" rpy="0.0  0.0  0.0"/>
+      <origin xyz="${BASE_LINE*0.5}  0.0  0.0" rpy="0.0  0.0  0.0"/>
     </joint>
     <link name="${camera}_right_link"/>

Commit message: Unify name with 'zedx'

File: vehicle/xacro/ai_car1.xacro (robot description, xacro)
@@ -11,5 +11,5 @@
   <xacro:property name="BASE_FOOTPRINT" value="base_footprint"/>
   <xacro:property name="BASE" value="base"/>
-  <xacro:property name="ZEDX" value="zedX"/>
+  <xacro:property name="ZEDX" value="zedx"/>
   <xacro:property name="WHEEL_LEFT" value="wheel_left"/>
   <xacro:property name="WHEEL_RIGHT" value="wheel_right"/>
@@ -22,5 +22,5 @@
     x="0.0" y="0.0" z="${WHEEL_RADIUS}"
     roll="0.0" pitch="0.0" yaw="${180.0*D2R}"/>
-  <!-- zedX -->
+  <!-- zedx -->
   <xacro:zed_joint_macro
     camera="${ZEDX}" parent="${BASE}"

Commit message: add launch and yaml, xacro for zedx camera

File: vehicle/xacro/ai_car1.xacro (robot description, xacro)
@@ -11,5 +11,5 @@
   <xacro:property name="BASE_FOOTPRINT" value="base_footprint"/>
   <xacro:property name="BASE" value="base"/>
-  <xacro:property name="ZEDX" value="zedx"/>
+  <xacro:property name="ZEDX" value="zed"/>
   <xacro:property name="WHEEL_LEFT" value="wheel_left"/>
   <xacro:property name="WHEEL_RIGHT" value="wheel_right"/>
@@ -26,9 +26,9 @@
     camera="${ZEDX}" parent="${BASE}"
     x="0.055" y="0.0" z="0.54"
-    roll="${(-90.0-2.0)*D2R}" pitch="0.0" yaw="${-90.0*D2R}"/>
+    roll="0.0" pitch="0.0" yaw="0.0"/>
   <xacro:zed_link_macro
     camera="${ZEDX}"
     size_x="0.132" size_y="0.020" size_z="0.006"
-    roll="0.0" pitch="0.0" yaw="0.0"/>
+    roll="${(-90.0-2.0)*D2R}" pitch="0.0" yaw="${-90.0*D2R}"/>
   <!-- wheel -->
   <xacro:wheel_joint_macro

File: vehicle/xacro/parts/zed_macro.xacro (robot description, xacro)
@@ -4,7 +4,7 @@
                params="camera parent
                        x y z roll pitch yaw">
-    <joint name="${camera}_joint" type="fixed">
+    <joint name="${camera}_camera_joint" type="fixed">
       <parent link="${parent}_link"/>
-      <child  link="${camera}_link"/>
+      <child  link="${camera}_camera_link"/>
       <origin xyz="${x} ${y} ${z}" rpy="${roll} ${pitch} ${yaw}"/>
     </joint>
@@ -14,7 +14,13 @@
                        size_x size_y size_z roll pitch yaw">
     <xacro:property name="MESH_FILE" value="package://vehicle/xacro/meshes/realsense_r200.dae"/>
-    <link name="${camera}_link">
+    <link name="${camera}_camera_link" />
+    <!-- Center frame -->
+    <joint name="${camera}_camera_center_joint" type="fixed">
+      <parent link="${camera}_camera_link"/>
+      <child link="${camera}_camera_center"/>
+    </joint>
+    <link name="${camera}_camera_center">
       <visual>
-        <origin xyz="${-size_x*0.5} ${-size_y*0.5} ${-size_z*0.5}" rpy="${roll} ${pitch} ${yaw}"/>
+        <origin xyz="${-size_x*0.5} ${-size_y*0.5} ${-size_z*0.5}" rpy="0.0 0.0 0.0"/>
         <geometry>
           <mesh filename="${MESH_FILE}"/>
@@ -22,5 +28,5 @@
       </visual>
       <collision>
-        <origin xyz="${-size_x*0.5} ${-size_y*0.5} ${-size_z*0.5}" rpy="${roll} ${pitch} ${yaw}"/>
+        <origin xyz="${-size_x*0.5} ${-size_y*0.5} ${-size_z*0.5}" rpy="0.0 0.0 0.0"/>
         <geometry>
           <box size="${size_x} ${size_y} ${size_z}"/>
@@ -28,17 +34,31 @@
       </collision>
     </link>
+    <!-- Left frame -->
     <xacro:property name="BASE_LINE" value="0.120005"/>
-    <joint name="${camera}_left_joint" type="fixed">
-      <parent link="${camera}_link"/>
-      <child link="${camera}_left_link"/>
-      <origin xyz="${-BASE_LINE*0.5}  0.0  0.0" rpy="0.0  0.0  0.0"/>
+    <joint name="${camera}_left_camera_joint" type="fixed">
+      <parent link="${camera}_camera_center"/>
+      <child link="${camera}_left_camera_frame"/>
+      <origin xyz="0.0 ${BASE_LINE*0.5}  0.0" rpy="0.0  0.0  0.0"/>
     </joint>
-    <link name="${camera}_left_link"/>
-    <joint name="${camera}_right_joint" type="fixed">
-      <parent link="${camera}_link"/>
-      <child link="${camera}_right_link"/>
-      <origin xyz="${BASE_LINE*0.5}  0.0  0.0" rpy="0.0  0.0  0.0"/>
+    <link name="${camera}_left_camera_frame" />
+    <joint name="${camera}_left_camera_optical_joint" type="fixed">
+      <parent link="${camera}_left_camera_frame"/>
+      <child link="${camera}_left_camera_optical_frame"/>
+      <origin xyz="0.0  0.0  0.0" rpy="${roll} ${pitch} ${yaw}"/>
     </joint>
-    <link name="${camera}_right_link"/>
+    <link name="${camera}_left_camera_optical_frame"/>
+    <!-- Right frame -->
+    <joint name="${camera}_right_camera_joint" type="fixed">
+      <parent link="${camera}_camera_center"/>
+      <child link="${camera}_right_camera_frame"/>
+      <origin xyz="0.0 ${-BASE_LINE*0.5} 0.0" rpy="0.0  0.0  0.0"/>
+    </joint>
+    <link name="${camera}_right_camera_frame"/>
+    <joint name="${camera}_right_camera_optical_joint" type="fixed">
+      <parent link="${camera}_right_camera_frame"/>
+      <child link="${camera}_right_camera_optical_frame"/>
+      <origin xyz="0.0  0.0  0.0" rpy="${roll} ${pitch} ${yaw}"/>
+    </joint>
+    <link name="${camera}_right_camera_optical_frame" />
   </xacro:macro>
 </robot>

Commit message: add stl config, fix launch yaml

File: vehicle/xacro/ai_car1.xacro (robot description, xacro)
@@ -29,6 +29,6 @@
   <xacro:zed_link_macro
     camera="${ZEDX}"
-    size_x="0.132" size_y="0.020" size_z="0.006"
-    roll="${(-90.0-2.0)*D2R}" pitch="0.0" yaw="${-90.0*D2R}"/>
+    size_x="0.035" size_y="0.16" size_z="0.03"
+    roll="${-90.0*D2R}" pitch="0.0" yaw="${-90.0*D2R}"/>
   <!-- wheel -->
   <xacro:wheel_joint_macro

File: vehicle/xacro/parts/zed_macro.xacro (robot description, xacro)
@@ -13,7 +13,8 @@
                params="camera
                        size_x size_y size_z roll pitch yaw">
-    <xacro:property name="MESH_FILE" value="package://vehicle/xacro/meshes/realsense_r200.dae"/>
+    <xacro:property name="MESH_FILE" value="package://vehicle/xacro/meshes/zedx.stl"/>
     <link name="${camera}_camera_link" />
     <!-- Center frame -->
+    <!-- camera_center_frame is used frame id for stereo camera -->
     <joint name="${camera}_camera_center_joint" type="fixed">
       <parent link="${camera}_camera_link"/>
@@ -22,5 +23,5 @@
     <link name="${camera}_camera_center">
       <visual>
-        <origin xyz="${-size_x*0.5} ${-size_y*0.5} ${-size_z*0.5}" rpy="0.0 0.0 0.0"/>
+        <origin xyz="0.0  0.0 ${-size_z*0.5}" rpy="0.0  0.0  0.0"/>
         <geometry>
           <mesh filename="${MESH_FILE}"/>
@@ -28,5 +29,5 @@
       </visual>
       <collision>
-        <origin xyz="${-size_x*0.5} ${-size_y*0.5} ${-size_z*0.5}" rpy="0.0 0.0 0.0"/>
+        <origin xyz="0.0  0.0 ${-size_z*0.5}" rpy="0.0  0.0  0.0"/>
         <geometry>
           <box size="${size_x} ${size_y} ${size_z}"/>

Commit message: Get zed extrinsic parameter from yaml in xacro.

File: vehicle/xacro/ai_car1.xacro (robot description, xacro)
@@ -15,4 +15,5 @@
   <xacro:property name="WHEEL_RIGHT" value="wheel_right"/>
   <xacro:property name="CASTER_BACK" value="caster_back"/>
+  <xacro:property name="ZED_SERIAL_NUMBER" value="SN48442725"/>
   <!-- base_footprint -->
   <link name="${BASE_FOOTPRINT}"/>
@@ -23,12 +24,6 @@
     roll="0.0" pitch="0.0" yaw="${180.0*D2R}"/>
   <!-- zedx -->
-  <xacro:zed_joint_macro
-    camera="${ZEDX}" parent="${BASE}"
-    x="0.055" y="0.0" z="0.54"
-    roll="0.0" pitch="0.0" yaw="0.0"/>
-  <xacro:zed_link_macro
-    camera="${ZEDX}"
-    size_x="0.035" size_y="0.16" size_z="0.03"
-    roll="${-90.0*D2R}" pitch="0.0" yaw="${-90.0*D2R}"/>
+  <xacro:zed_macro
+    camera="${ZEDX}" parent="${BASE}" zed_serial_number="${ZED_SERIAL_NUMBER}"/>
   <!-- wheel -->
   <xacro:wheel_joint_macro

File: vehicle/xacro/parts/zed_macro.xacro (robot description, xacro)
@@ -1,20 +1,19 @@
 <?xml version="1.0" ?>
 <robot xmlns:xacro="http://www.ros.org/wiki/xacro">
-  <xacro:macro name="zed_joint_macro"
-               params="camera parent
-                       x y z roll pitch yaw">
+  <xacro:macro name="zed_macro"
+               params="camera parent zed_serial_number">
+    <xacro:property name="ZED_PARAM_YAML_PATH" value="$(find vehicle)/config/zedx/camera_params/${zed_serial_number}/extrinsic.yaml" />
+    <xacro:property name="POSISION" value="${load_yaml(ZED_PARAM_YAML_PATH)['position']}" />
+    <xacro:property name="ORIENTATION" value="${load_yaml(ZED_PARAM_YAML_PATH)['orientation']}" />
+    <xacro:property name="MESH_FILE" value="package://vehicle/xacro/meshes/zedx.stl"/>
+    <xacro:property name="SIZE" value="${dict(x=0.035, y=0.16, z=0.03)}"/>
+    <xacro:property name="BASE_LINE" value="0.120005"/>
     <joint name="${camera}_camera_joint" type="fixed">
       <parent link="${parent}_link"/>
       <child  link="${camera}_camera_link"/>
-      <origin xyz="${x} ${y} ${z}" rpy="${roll} ${pitch} ${yaw}"/>
+      <origin xyz="${POSISION['x']} ${POSISION['y']} ${POSISION['z']}" rpy="0.0  0.0  0.0"/>
     </joint>
-  </xacro:macro>
-  <xacro:macro name="zed_link_macro"
-               params="camera
-                       size_x size_y size_z roll pitch yaw">
-    <xacro:property name="MESH_FILE" value="package://vehicle/xacro/meshes/zedx.stl"/>
     <link name="${camera}_camera_link" />
-    <!-- Center frame -->
-    <!-- camera_center_frame is used in frame id for stereo camera -->
+    <!-- Center frame (is used in frame_id for stereo camera)-->
     <joint name="${camera}_camera_center_joint" type="fixed">
       <parent link="${camera}_camera_link"/>
@@ -23,5 +22,5 @@
     <link name="${camera}_camera_center">
       <visual>
-        <origin xyz="0.0  0.0 ${-size_z*0.5}" rpy="0.0  0.0  0.0"/>
+        <origin xyz="0.0  0.0 ${-SIZE['z']*0.5}" rpy="0.0  0.0  0.0"/>
         <geometry>
           <mesh filename="${MESH_FILE}"/>
@@ -29,12 +28,11 @@
       </visual>
       <collision>
-        <origin xyz="0.0  0.0 ${-size_z*0.5}" rpy="0.0  0.0  0.0"/>
+        <origin xyz="0.0  0.0 ${-SIZE['z']*0.5}" rpy="0.0  0.0  0.0"/>
         <geometry>
-          <box size="${size_x} ${size_y} ${size_z}"/>
+          <box size="${SIZE['x']} ${SIZE['y']} ${SIZE['z']}"/>
         </geometry>
       </collision>
     </link>
     <!-- Left frame -->
-    <xacro:property name="BASE_LINE" value="0.120005"/>
     <joint name="${camera}_left_camera_joint" type="fixed">
       <parent link="${camera}_camera_center"/>
@@ -46,5 +44,6 @@
       <parent link="${camera}_left_camera_frame"/>
       <child link="${camera}_left_camera_optical_frame"/>
-      <origin xyz="0.0  0.0  0.0" rpy="${roll} ${pitch} ${yaw}"/>
+      <origin xyz="0.0  0.0  0.0"
+              rpy="${ORIENTATION['r']*D2R} ${ORIENTATION['p']*D2R} ${ORIENTATION['y']*D2R}"/>
     </joint>
     <link name="${camera}_left_camera_optical_frame"/>
@@ -59,5 +58,6 @@
       <parent link="${camera}_right_camera_frame"/>
       <child link="${camera}_right_camera_optical_frame"/>
-      <origin xyz="0.0  0.0  0.0" rpy="${roll} ${pitch} ${yaw}"/>
+      <origin xyz="0.0  0.0  0.0"
+              rpy="${ORIENTATION['r']*D2R} ${ORIENTATION['p']*D2R} ${ORIENTATION['y']*D2R}"/>
     </joint>
     <link name="${camera}_right_camera_optical_frame" />

Commit message: sort folder and modified xacro yaml

File: vehicle/xacro/ai_car1.xacro (robot description, xacro)
@@ -15,5 +15,4 @@
   <xacro:property name="WHEEL_RIGHT" value="wheel_right"/>
   <xacro:property name="CASTER_BACK" value="caster_back"/>
-  <xacro:property name="ZED_SERIAL_NUMBER" value="SN48442725"/>
   <!-- base_footprint -->
   <link name="${BASE_FOOTPRINT}"/>
@@ -25,5 +24,5 @@
   <!-- zedx -->
   <xacro:zed_macro
-    camera="${ZEDX}" parent="${BASE}" zed_serial_number="${ZED_SERIAL_NUMBER}"/>
+    camera="${ZEDX}" parent="${BASE}"/>
   <!-- wheel -->
   <xacro:wheel_joint_macro

File: vehicle/xacro/parts/zed_macro.xacro (robot description, xacro)
@@ -2,6 +2,6 @@
 <robot xmlns:xacro="http://www.ros.org/wiki/xacro">
   <xacro:macro name="zed_macro"
-               params="camera parent zed_serial_number">
-    <xacro:property name="ZED_PARAM_YAML_PATH" value="$(find vehicle)/config/zedx/camera_params/${zed_serial_number}/extrinsic.yaml" />
+               params="camera parent">
+    <xacro:property name="ZED_PARAM_YAML_PATH" value="$(find vehicle)/config/zedx/extrinsic/extrinsic.yaml" />
     <xacro:property name="POSITION" value="${load_yaml(ZED_PARAM_YAML_PATH)['position']}" />
     <xacro:property name="ORIENTATION" value="${load_yaml(ZED_PARAM_YAML_PATH)['orientation']}" />

Commit message: Add feature to switch wheel-related TF publishing between `/tf` and `/tf_static`.

File: vehicle/xacro/ai_car1.xacro (robot description, xacro)
@@ -15,4 +15,5 @@
   <xacro:property name="WHEEL_RIGHT" value="wheel_right"/>
   <xacro:property name="CASTER_BACK" value="caster_back"/>
+  <xacro:property name="WHEEL_JOINT_TYPE" value="fixed"/>
   <!-- base_footprint -->
   <link name="${BASE_FOOTPRINT}"/>
@@ -28,4 +29,5 @@
   <xacro:wheel_joint_macro
     wheel="${WHEEL_LEFT}" parent="${BASE}"
+    joint_type="${WHEEL_JOINT_TYPE}"
     x="0.0" y="0.3" z="${WHEEL_RADIUS}"
     roll="${90.0*D2R}" pitch="0.0" yaw="${90.0*D2R}"/>
@@ -36,4 +38,5 @@
   <xacro:wheel_joint_macro
     wheel="${WHEEL_RIGHT}" parent="${BASE}"
+    joint_type="${WHEEL_JOINT_TYPE}"
     x="0.0" y="-0.3" z="${WHEEL_RADIUS}"
     roll="${90.0*D2R}" pitch="0.0" yaw="${90.0*D2R}"/>
@@ -45,4 +48,5 @@
   <xacro:caster_back_joint_macro
     caster_back="${CASTER_BACK}" parent="${BASE}"
+    joint_type="${WHEEL_JOINT_TYPE}"
     x="-0.76" y="0.0" z="${CASTER_RADIUS}"
     roll="${90.0*D2R}" pitch="0.0" yaw="${90.0*D2R}"/>

File: vehicle/xacro/parts/caster_back_macro.xacro (robot description, xacro)
@@ -2,7 +2,7 @@
 <robot xmlns:xacro="http://www.ros.org/wiki/xacro">
   <xacro:macro name="caster_back_joint_macro"
-               params="caster_back parent
+               params="caster_back parent joint_type
                        x y z roll pitch yaw">
-    <joint name="${caster_back}_joint" type="continuous">
+    <joint name="${caster_back}_joint" type="${joint_type}">
       <parent link="${parent}_link"/>
       <child  link="${caster_back}_link"/>

File: vehicle/xacro/parts/wheel_macro.xacro (robot description, xacro)
@@ -2,7 +2,7 @@
 <robot xmlns:xacro="http://www.ros.org/wiki/xacro">
   <xacro:macro name="wheel_joint_macro"
-               params="wheel parent
+               params="wheel parent joint_type
                        x y z roll pitch yaw">
-    <joint name="${wheel}_joint" type="continuous">
+    <joint name="${wheel}_joint" type="${joint_type}">
       <parent link="${parent}_link"/>
       <child  link="${wheel}_link"/>
