Commit message: Revert changes related to tf.

File: vehicle/xacro/ai_car1.xacro (robot description, xacro)
@@ -15,5 +15,4 @@
   <xacro:property name="WHEEL_RIGHT" value="wheel_right"/>
   <xacro:property name="CASTER_BACK" value="caster_back"/>
-  <xacro:property name="WHEEL_JOINT_TYPE" value="fixed"/>
   <!-- base_footprint -->
   <link name="${BASE_FOOTPRINT}"/>
@@ -29,5 +28,4 @@
   <xacro:wheel_joint_macro
     wheel="${WHEEL_LEFT}" parent="${BASE}"
-    joint_type="${WHEEL_JOINT_TYPE}"
     x="0.0" y="0.3" z="${WHEEL_RADIUS}"
     roll="${90.0*D2R}" pitch="0.0" yaw="${90.0*D2R}"/>
@@ -38,5 +36,4 @@
   <xacro:wheel_joint_macro
     wheel="${WHEEL_RIGHT}" parent="${BASE}"
-    joint_type="${WHEEL_JOINT_TYPE}"
     x="0.0" y="-0.3" z="${WHEEL_RADIUS}"
     roll="${90.0*D2R}" pitch="0.0" yaw="${90.0*D2R}"/>
@@ -48,5 +45,4 @@
   <xacro:caster_back_joint_macro
     caster_back="${CASTER_BACK}" parent="${BASE}"
-    joint_type="${WHEEL_JOINT_TYPE}"
     x="-0.76" y="0.0" z="${CASTER_RADIUS}"
     roll="${90.0*D2R}" pitch="0.0" yaw="${90.0*D2R}"/>

File: vehicle/xacro/parts/caster_back_macro.xacro (robot description, xacro)
@@ -2,7 +2,7 @@
 <robot xmlns:xacro="http://www.ros.org/wiki/xacro">
   <xacro:macro name="caster_back_joint_macro"
-               params="caster_back parent joint_type
+               params="caster_back parent
                        x y z roll pitch yaw">
-    <joint name="${caster_back}_joint" type="${joint_type}">
+    <joint name="${caster_back}_joint" type="continuous">
       <parent link="${parent}_link"/>
       <child  link="${caster_back}_link"/>

File: vehicle/xacro/parts/wheel_macro.xacro (robot description, xacro)
@@ -2,7 +2,7 @@
 <robot xmlns:xacro="http://www.ros.org/wiki/xacro">
   <xacro:macro name="wheel_joint_macro"
-               params="wheel parent joint_type
+               params="wheel parent
                        x y z roll pitch yaw">
-    <joint name="${wheel}_joint" type="${joint_type}">
+    <joint name="${wheel}_joint" type="continuous">
       <parent link="${parent}_link"/>
       <child  link="${wheel}_link"/>
