Commit message: Update how to load yaml.

File: sample_vehicle/xacro/parts/zed_macro.xacro (robot description, xacro)
@@ -4,6 +4,6 @@
                params="camera parent">
     <xacro:property name="ZED_PARAM_YAML_PATH" value="$(find sample_vehicle)/config/zedx/extrinsic/extrinsic.yaml" />
-    <xacro:property name="POSITION" value="${load_yaml(ZED_PARAM_YAML_PATH)['position']}" />
-    <xacro:property name="ORIENTATION" value="${load_yaml(ZED_PARAM_YAML_PATH)['orientation']}" />
+    <xacro:property name="POSITION" value="${xacro.load_yaml(ZED_PARAM_YAML_PATH)['position']}" />
+    <xacro:property name="ORIENTATION" value="${xacro.load_yaml(ZED_PARAM_YAML_PATH)['orientation']}" />
     <xacro:property name="MESH_FILE" value="package://sample_vehicle/xacro/meshes/zedx.stl"/>
     <xacro:property name="SIZE" value="${dict(x=0.035, y=0.16, z=0.03)}"/>

Commit message: Revert YAML loading method due to incompatibility with foxy.

File: sample_vehicle/xacro/parts/zed_macro.xacro (robot description, xacro)
@@ -4,6 +4,6 @@
                params="camera parent">
     <xacro:property name="ZED_PARAM_YAML_PATH" value="$(find sample_vehicle)/config/zedx/extrinsic/extrinsic.yaml" />
-    <xacro:property name="POSITION" value="${xacro.load_yaml(ZED_PARAM_YAML_PATH)['position']}" />
-    <xacro:property name="ORIENTATION" value="${xacro.load_yaml(ZED_PARAM_YAML_PATH)['orientation']}" />
+    <xacro:property name="POSITION" value="${load_yaml(ZED_PARAM_YAML_PATH)['position']}" />
+    <xacro:property name="ORIENTATION" value="${load_yaml(ZED_PARAM_YAML_PATH)['orientation']}" />
     <xacro:property name="MESH_FILE" value="package://sample_vehicle/xacro/meshes/zedx.stl"/>
     <xacro:property name="SIZE" value="${dict(x=0.035, y=0.16, z=0.03)}"/>
